File: Power mangement.kicad_pcb (KiCad board)
At the start: 4 copper layers, 92.2 x 53 mm, 28 parts, among them Q1 FDS6890A, U1 max1954eub+T, U2 TB004-508-02BE, U3 TB004-508-02BE, U4 MBRS340T3G, U5 TB004-508-02BE

Commit message: PCB layout change placement
Parts:
- removed the C3 at (143.0, 102.3)
- moved C4 54.5 mm to (137.4, 79.8)
- moved R4 44.2 mm to (138.1, 99.2), turned to -90 degrees
- moved C5 42.3 mm to (142.1, 93.5), turned to 90 degrees
- moved C3 30.8 mm to (142.7, 102.8), turned to 90 degrees
- moved R3 27.1 mm to (139.6, 99.2), turned to 90 degrees
- moved R2 26.9 mm to (149.3, 102.8), turned to -90 degrees
- moved C7 23.7 mm to (151.5, 102.9), turned to -90 degrees
Routing:
- added copper zone on In1.Cu, net GND
- removed copper zone on F.Cu, net P12V
- removed copper zone on F.Cu, net P5V
